File: Other Versions/GSM-Parakeet/parakeet_board.sch (EAGLE design)
At the start: 14 parts, among them IC1 TP4056

Commit message: Updated GSM version
Parts:
- removed U$2: SIM800L_GSM_MODULE, SIM800L Module:SIM800L_GSM_MODULE
- added SIM800L: SIM800L_PARAKEET_ONLY, SIM800L Module:SIM800L_PARAKEET_ONLY
- C1, C2: value 10uf -> 10μf
- R2, R3: value 1K -> 150Ω
- R_PROG: value 1.2K=1A -> 1.2KΩ=1A
- renumbered IC1 to TP4056, U$1 to USB, U$3 to SWITCH, U$4 to WIXEL
Connections:
- net GND: now also SIM800L.P$6_GND; no longer U$2.P$6_GND
- net N$12: now also SIM800L.P$2_VIN; no longer U$2.P$1
- net N$13: now also SIM800L.P$8_DTR; no longer U$2.P$8_DTR
- net N$2: now also SIM800L.P$5_TXD; no longer U$2.P$5_TXD
- net N$9: now also SIM800L.P$4_RXD; no longer U$2.P$4_RXD

Commit message: Updated GSM version
Changed lines of the file:
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@@
 <part name="GND1" library="SparkFun-Aesthetics" deviceset="GND" device=""/>
 <part name="GND2" library="SparkFun-Aesthetics" deviceset="GND" device=""/>
-<part name="GND3" library="SparkFun-Aesthetics" deviceset="GND" device=""/>
 <part name="GND4" library="SparkFun-Aesthetics" deviceset="GND" device=""/>
 <part name="WIXEL" library="wixel" deviceset="WIXEL_PARAKEET_ONLY" device=""/>
@@
 <instance part="JST2" gate="G$1" x="101.6" y="48.26" rot="R180"/>
 <instance part="SWITCH" gate="MSK-12C02" x="102.87" y="60.96"/>
-<instance part="GND1" gate="1" x="109.22" y="71.12" rot="R180"/>
-<instance part="GND2" gate="1" x="134.62" y="71.12" rot="R180"/>
-<instance part="GND3" gate="1" x="134.62" y="15.24"/>
-<instance part="GND4" gate="1" x="139.7" y="15.24"/>
+<instance part="GND1" gate="1" x="109.22" y="68.58" rot="R180"/>
+<instance part="GND2" gate="1" x="134.62" y="68.58" rot="R180"/>
+<instance part="GND4" gate="1" x="139.7" y="25.4"/>
 <instance part="WIXEL" gate="G$1" x="121.92" y="40.64"/>
 <instance part="SIM800L" gate="G$1" x="157.48" y="40.64"/>
@@
 <segment>
 <pinref part="GND1" gate="1" pin="GND"/>
-<wire x1="109.22" y1="68.58" x2="109.22" y2="58.42" width="0.1524" layer="91"/>
+<wire x1="109.22" y1="66.04" x2="109.22" y2="58.42" width="0.1524" layer="91"/>
 <pinref part="WIXEL" gate="G$1" pin="P$1-GND1"/>
 </segment>
 <segment>
 <pinref part="GND2" gate="1" pin="GND"/>
-<wire x1="134.62" y1="68.58" x2="134.62" y2="58.42" width="0.1524" layer="91"/>
+<wire x1="134.62" y1="66.04" x2="134.62" y2="58.42" width="0.1524" layer="91"/>
 <pinref part="WIXEL" gate="G$1" pin="P$12-GND2"/>
 </segment>
 <segment>
-<pinref part="GND3" gate="1" pin="GND"/>
-<wire x1="134.62" y1="17.78" x2="134.62" y2="30.48" width="0.1524" layer="91"/>
 <pinref part="WIXEL" gate="G$1" pin="P$23-GND3"/>
-</segment>
-<segment>
 <pinref part="GND4" gate="1" pin="GND"/>
-<wire x1="139.7" y1="17.78" x2="139.7" y2="35.56" width="0.1524" layer="91"/>
 <pinref part="SIM800L" gate="G$1" pin="P$6_GND"/>
+<wire x1="139.7" y1="27.94" x2="139.7" y2="30.48" width="0.1524" layer="91"/>
+<wire x1="139.7" y1="30.48" x2="139.7" y2="35.56" width="0.1524" layer="91"/>
+<wire x1="134.62" y1="30.48" x2="139.7" y2="30.48" width="0.1524" layer="91"/>
+<junction x="139.7" y="30.48"/>
 </segment>
 </net>

Commit message: Updated GSM Version
Parts:
- R_PROG: value 1.2KΩ=1A -> 1.2KΩ
Changed lines of the file:
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@@
 <part name="TP4056" library="TP4056" deviceset="TP4056" device=""/>
 <part name="USB" library="micro usb B - sparkfun - china - hole 4LEGS TEST" deviceset="MICRO-USB-B" device=""/>
-<part name="R_PROG" library="resistor" deviceset="R-EU_" device="R1206" value="1.2KΩ=1A"/>
+<part name="R_PROG" library="resistor" deviceset="R-EU_" device="R1206" value="1.2KΩ"/>
 <part name="C1" library="resistor" deviceset="C-EU" device="C1206" value="10μf"/>
 <part name="LED1" library="led" deviceset="LED" device="CHIPLED_1206" value="RED"/>

Commit message: Updated GSM Version
Parts:
- removed R3: 150Ω, resistor:R-EU_R1206
- added R1: 330Ω, resistor:R-EU_R1206
- R2: value 150Ω -> 330Ω
Connections:
- net GND: now also TP4056.GND_PAD
- net N$3: now also R1.2; no longer R2.2
- net N$4: now also R2.2; no longer R3.2
- net N$5: now also R1.1; no longer R2.1
- net N$6: now also R2.1; no longer R3.1
Other:
- moved on the sheet: C2, R2, R_PROG
Changed lines of the file:
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@@
 <part name="LED1" library="led" deviceset="LED" device="CHIPLED_1206" value="RED"/>
 <part name="LED2" library="led" deviceset="LED" device="CHIPLED_1206" value="GREEN"/>
-<part name="R2" library="resistor" deviceset="R-EU_" device="R1206" value="150Ω"/>
-<part name="R3" library="resistor" deviceset="R-EU_" device="R1206" value="150Ω"/>
+<part name="R1" library="resistor" deviceset="R-EU_" device="R1206" value="330Ω"/>
+<part name="R2" library="resistor" deviceset="R-EU_" device="R1206" value="330Ω"/>
 <part name="C2" library="resistor" deviceset="C-EU" device="C1206" value="10μf"/>
 <part name="+" library="SparkFun-Connectors" deviceset="M02" device="PTH" value="BAT"/>
@@
 <sheet>
 <plain>
-<text x="-30.48" y="25.4" size="1.778" layer="91">RPROG -     IBAT
+<text x="-22.86" y="40.64" size="1.778" layer="91" align="center">RPROG -     IBAT
 (k)        -    (mA)
 10         -    130
@@
 </plain>
 <instances>
-<instance part="TP4056" gate="G$1" x="40.64" y="48.26"/>
-<instance part="USB" gate="G$1" x="2.54" y="40.64"/>
-<instance part="R_PROG" gate="G$1" x="27.94" y="43.18"/>
+<instance part="TP4056" gate="G$1" x="46.99" y="41.91"/>
+<instance part="USB" gate="G$1" x="-2.54" y="40.64"/>
+<instance part="R_PROG" gate="G$1" x="22.86" y="43.18"/>
 <instance part="C1" gate="G$1" x="60.96" y="30.48" rot="R270"/>
 <instance part="LED1" gate="G$1" x="83.82" y="45.72" rot="R270"/>
 <instance part="LED2" gate="G$1" x="83.82" y="38.1" rot="R270"/>
-<instance part="R2" gate="G$1" x="71.12" y="45.72"/>
-<instance part="R3" gate="G$1" x="71.12" y="38.1"/>
-<instance part="C2" gate="G$1" x="27.94" y="35.56"/>
+<instance part="R1" gate="G$1" x="71.12" y="45.72"/>
+<instance part="R2" gate="G$1" x="71.12" y="38.1"/>
+<instance part="C2" gate="G$1" x="22.86" y="35.56"/>
 <instance part="+" gate="G$1" x="101.6" y="33.02" rot="R180"/>
 <instance part="JST2" gate="G$1" x="101.6" y="48.26" rot="R180"/>
@@
 <pinref part="TP4056" gate="G$1" pin="PROG"/>
 <pinref part="R_PROG" gate="G$1" pin="2"/>
-<wire x1="33.02" y1="43.18" x2="35.56" y2="43.18" width="0.1524" layer="91"/>
+<wire x1="27.94" y1="43.18" x2="30.48" y2="43.18" width="0.1524" layer="91"/>
 </segment>
 </net>
 <net name="GND" class="0">
 <segment>
-<wire x1="20.32" y1="30.48" x2="20.32" y2="40.64" width="0.1524" layer="91"/>
+<wire x1="15.24" y1="30.48" x2="15.24" y2="40.64" width="0.1524" layer="91"/>
 <pinref part="TP4056" gate="G$1" pin="GND"/>
-<wire x1="20.32" y1="40.64" x2="35.56" y2="40.64" width="0.1524" layer="91"/>
+<wire x1="15.24" y1="40.64" x2="30.48" y2="40.64" width="0.1524" layer="91"/>
 <pinref part="TP4056" gate="G$1" pin="TEMP"/>
-<wire x1="35.56" y1="45.72" x2="20.32" y2="45.72" width="0.1524" layer="91"/>
-<wire x1="20.32" y1="45.72" x2="20.32" y2="43.18" width="0.1524" layer="91"/>
-<junction x="20.32" y="40.64"/>
+<wire x1="30.48" y1="45.72" x2="15.24" y2="45.72" width="0.1524" layer="91"/>
+<wire x1="15.24" y1="45.72" x2="15.24" y2="43.18" width="0.1524" layer="91"/>
+<junction x="15.24" y="40.64"/>
 <pinref part="R_PROG" gate="G$1" pin="1"/>
-<wire x1="20.32" y1="43.18" x2="20.32" y2="40.64" width="0.1524" layer="91"/>
-<wire x1="22.86" y1="43.18" x2="20.32" y2="43.18" width="0.1524" layer="91"/>
-<junction x="20.32" y="43.18"/>
+<wire x1="15.24" y1="43.18" x2="15.24" y2="40.64" width="0.1524" layer="91"/>
+<wire x1="17.78" y1="43.18" x2="15.24" y2="43.18" width="0.1524" layer="91"/>
+<junction x="15.24" y="43.18"/>
 <pinref part="C2" gate="G$1" pin="2"/>
-<wire x1="27.94" y1="30.48" x2="20.32" y2="30.48" width="0.1524" layer="91"/>
+<wire x1="22.86" y1="30.48" x2="15.24" y2="30.48" width="0.1524" layer="91"/>
 <pinref part="C1" gate="G$1" pin="2"/>
-<wire x1="27.94" y1="30.48" x2="55.88" y2="30.48" width="0.1524" layer="91"/>
+<wire x1="22.86" y1="30.48" x2="46.99" y2="30.48" width="0.1524" layer="91"/>
 <pinref part="USB" gate="G$1" pin="GND"/>
-<wire x1="17.78" y1="30.48" x2="20.32" y2="30.48" width="0.1524" layer="91"/>
-<junction x="20.32" y="30.48"/>
+<wire x1="46.99" y1="30.48" x2="55.88" y2="30.48" width="0.1524" layer="91"/>
+<wire x1="12.7" y1="30.48" x2="15.24" y2="30.48" width="0.1524" layer="91"/>
+<junction x="15.24" y="30.48"/>
 <wire x1="91.44" y1="25.4" x2="55.88" y2="25.4" width="0.1524" layer="91"/>
 <wire x1="55.88" y1="25.4" x2="55.88" y2="30.48" width="0.1524" layer="91"/>
@@
 <wire x1="93.98" y1="30.48" x2="91.44" y2="30.48" width="0.1524" layer="91"/>
 <junction x="91.44" y="30.48"/>
-<junction x="27.94" y="30.48"/>
+<junction x="22.86" y="30.48"/>
+<pinref part="TP4056" gate="G$1" pin="GND_PAD"/>
+<junction x="46.99" y="30.48"/>
 </segment>
 <segment>
@@
 <segment>
 <pinref part="LED1" gate="G$1" pin="C"/>
-<pinref part="R2" gate="G$1" pin="2"/>
+<pinref part="R1" gate="G$1" pin="2"/>
 <wire x1="76.2" y1="45.72" x2="78.74" y2="45.72" width="0.1524" layer="91"/>
 </segment>
@@
 <segment>
 <pinref part="LED2" gate="G$1" pin="C"/>
-<pinref part="R3" gate="G$1" pin="2"/>
+<pinref part="R2" gate="G$1" pin="2"/>
 <wire x1="76.2" y1="38.1" x2="78.74" y2="38.1" width="0.1524" layer="91"/>
 </segment>
@@
 <segment>
 <pinref part="TP4056" gate="G$1" pin="CHRG"/>
-<pinref part="R2" gate="G$1" pin="1"/>
+<pinref part="R1" gate="G$1" pin="1"/>
 <wire x1="63.5" y1="43.18" x2="66.04" y2="43.18" width="0.1524" layer="91"/>
 <wire x1="66.04" y1="43.18" x2="66.04" y2="45.72" width="0.1524" layer="91"/>
@@
 <segment>
 <pinref part="TP4056" gate="G$1" pin="STDBY"/>
-<pinref part="R3" gate="G$1" pin="1"/>
+<pinref part="R2" gate="G$1" pin="1"/>
 <wire x1="63.5" y1="40.64" x2="66.04" y2="40.64" width="0.1524" layer="91"/>
 <wire x1="66.04" y1="40.64" x2="66.04" y2="38.1" width="0.1524" layer="91"/>
@@
 <segment>
 <pinref part="USB" gate="G$1" pin="VCC"/>
-<wire x1="17.78" y1="50.8" x2="27.94" y2="50.8" width="0.1524" layer="91"/>
-<wire x1="27.94" y1="50.8" x2="63.5" y2="50.8" width="0.1524" layer="91"/>
+<wire x1="12.7" y1="50.8" x2="22.86" y2="50.8" width="0.1524" layer="91"/>
+<wire x1="22.86" y1="50.8" x2="63.5" y2="50.8" width="0.1524" layer="91"/>
 <wire x1="63.5" y1="50.8" x2="86.36" y2="50.8" width="0.1524" layer="91"/>
 <wire x1="86.36" y1="50.8" x2="86.36" y2="45.72" width="0.1524" layer="91"/>
@@
 <wire x1="86.36" y1="45.72" x2="86.36" y2="38.1" width="0.1524" layer="91"/>
 <pinref part="TP4056" gate="G$1" pin="VCC"/>
-<wire x1="35.56" y1="38.1" x2="27.94" y2="38.1" width="0.1524" layer="91"/>
-<wire x1="27.94" y1="38.1" x2="27.94" y2="50.8" width="0.1524" layer="91"/>
-<junction x="27.94" y="50.8"/>
+<wire x1="30.48" y1="38.1" x2="22.86" y2="38.1" width="0.1524" layer="91"/>
+<wire x1="22.86" y1="38.1" x2="22.86" y2="50.8" width="0.1524" layer="91"/>
+<junction x="22.86" y="50.8"/>
 <pinref part="TP4056" gate="G$1" pin="CE"/>
 <wire x1="63.5" y1="45.72" x2="63.5" y2="50.8" width="0.1524" layer="91"/>
 <junction x="63.5" y="50.8"/>
 <pinref part="C2" gate="G$1" pin="1"/>
-<junction x="27.94" y="38.1"/>
+<junction x="22.86" y="38.1"/>
 <junction x="86.36" y="45.72"/>
 </segment>
