File: Other Versions/GSM-Parakeet/parakeet_board.brd (EAGLE design)
At the start: 35 x 38.5 mm, 14 parts, among them IC1 TP4056

Commit message: Updated GSM version
Parts:
- removed IC1: TP4056, TP4056:SOP-8
- removed U$2: SIM800L_GSM_MODULE, SIM800L Module:SIM800L_GSM_MODULE
- removed U$3: MSK-12C02_SMD_SPDT_SWITCH, MSK-12C02 SMD Micro Slider Switch SPDT:MSK-12C02
- added SIM800L: SIM800L_PARAKEET_ONLY, SIM800L Module:SIM800L_PARAKEET_ONLY
- added SWITCH: MSK-12C02_SMD_SPDT_SWITCH, MSK-12C02 SMD Micro Slider Switch SPDT:MSK-12C02
- added TP4056: TP4056, TP4056:SOP-8
- added USB: MICRO-USB-B, micro usb B - sparkfun - china - hole 4LEGS TEST:MICRO_USB_4_LEGS
- C1, C2: value 10uf -> 10μf
- R2, R3: value 1K -> 150Ω
- R_PROG: value 1.2K=1A -> 1.2KΩ=1A
- U$1: value MICRO-USB-B -> (none); device micro usb B - sparkfun - china - hole 4LEGS TEST:MICRO_USB_4_LEGS -> LOGO:PARAKEET_VECTOR
- moved C2 28.9 mm to (2.10, 62.2), flipped to the top, turned to 90 degrees
- moved U$1 27.2 mm to (8.89, 54.6), turned to 0 degrees
- moved LED1 22.8 mm to (33.4, 70.3)
- moved LED2 22.6 mm to (33.4, 64.5)
- moved R3 22.0 mm to (33.5, 55.0), flipped to the top, turned to 90 degrees
- moved R2 16.2 mm to (30.5, 75.4), turned to 180 degrees
- moved R_PROG 13.7 mm to (4.83, 56.8), flipped to the top, turned to 0 degrees
- moved JST2 10.7 mm to (8.64, 46.9), flipped to the top
- moved C1 8.22 mm to (9.33, 73.0), flipped to the top
- moved + 3.28 mm to (2.03, 73.6)
- renumbered U$4 to WIXEL
Connections:
- net GND: now also SIM800L.P$6_GND, TP4056.1, TP4056.3, USB.GND; no longer IC1.1, IC1.3, U$1.GND, U$2.P$6_GND
- net N$1: now also TP4056.2; no longer IC1.2
- net N$12: now also SIM800L.P$2_VIN, SWITCH.L1; no longer U$2.P$1, U$3.L1
- net N$13: now also SIM800L.P$8_DTR; no longer U$2.P$8_DTR
- net N$2: now also SIM800L.P$5_TXD; no longer U$2.P$5_TXD
- net N$5: now also TP4056.7; no longer IC1.7
- net N$6: now also TP4056.6; no longer IC1.6
- net N$7: now also TP4056.4, TP4056.8, USB.VCC; no longer IC1.4, IC1.8, U$1.VCC
- net N$8: now also SWITCH.COM, TP4056.5; no longer IC1.5, U$3.COM
- net N$9: now also SIM800L.P$4_RXD; no longer U$2.P$4_RXD
Routing:
- net N$5: track 11.4 -> 52.4 mm, vias 0 -> 3
- net N$6: track 6.61 -> 45.0 mm, vias 0 -> 2
- net N$7: track 42.2 -> 64.9 mm, vias 3 -> 1
- net N$9: track 7.41 -> 23.6 mm
- net N$2: track 6.45 -> 21.8 mm, vias 0 -> 1
- net N$8: track 36.6 -> 52.0 mm, vias 0 -> 1
- net N$13: track 24.8 -> 10.4 mm
- net N$12: track 37.7 -> 23.8 mm
- net N$3: track 12.6 -> 6.02 mm
- net N$1: track 7.13 -> 3.32 mm
- net N$4: track 9.10 -> 8.15 mm, vias 1 -> 0
- added copper zone on layer 16, net N$10
- added copper zone on layer 1, net N$11
Other:
- board size 35 x 38.5 mm -> 35 x 38.4 mm
- board text added: "12-Jun-2016 Rev.02"

Commit message: Updated GSM version
Other:
- board text added: "12-Jun-2016 Rev.03"
- board text added: "OFF"
- board text added: "ON"
- board text removed: "12-Jun-2016 Rev.02"
Changed lines of the file:
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@@
 <hole x="2.0955" y="78.2955" drill="1.5"/>
 <text x="23.0505" y="59.7535" size="1.4224" layer="25" rot="R270" align="center">12-Jun-2016
-Rev.02</text>
+Rev.03</text>
+<text x="13.081" y="75.438" size="1.778" layer="25" rot="R90">ON</text>
+<text x="5.6515" y="74.422" size="1.778" layer="25" rot="R90">OFF</text>
 </plain>
 <attributes>
@@
 <contactref element="+" pad="1"/>
 <contactref element="SWITCH" pad="COM"/>
-<via x="4.445" y="50.8" extent="1-16" drill="0.6"/>
+<via x="3.683" y="51.562" extent="1-16" drill="0.6"/>
 <wire x1="4.2545" y1="71.882" x2="2.54" y2="73.5965" width="0.6096" layer="16"/>
 <wire x1="2.54" y1="73.5965" x2="2.032" y2="73.5965" width="0.4064" layer="16"/>
-<wire x1="4.445" y1="50.8" x2="7.399" y2="50.8" width="0.6096" layer="1"/>
 <wire x1="7.399" y1="50.8" x2="7.636" y2="50.563" width="0.4064" layer="1"/>
 <wire x1="2.032" y1="73.5965" x2="8.0645" y2="73.5965" width="0.6096" layer="16"/>
@@
 <wire x1="4.2545" y1="71.882" x2="4.2545" y2="69.9135" width="0.6096" layer="16"/>
 <wire x1="4.2545" y1="69.9135" x2="2.8575" y2="68.5165" width="0.6096" layer="16"/>
-<wire x1="4.445" y1="50.8" x2="2.8575" y2="52.3875" width="0.6096" layer="16"/>
 <wire x1="2.8575" y1="52.3875" x2="2.8575" y2="68.5165" width="0.6096" layer="16"/>
 <wire x1="7.9345" y1="73.025" x2="8.4455" y2="73.025" width="0.6096" layer="1"/>
@@
 <wire x1="7.9345" y1="73.025" x2="7.363" y2="73.5965" width="0.6096" layer="1"/>
 <wire x1="7.363" y1="73.5965" x2="2.032" y2="73.5965" width="0.6096" layer="1"/>
+<wire x1="2.8575" y1="52.3875" x2="3.683" y2="51.562" width="0.6096" layer="16"/>
+<wire x1="7.399" y1="50.8" x2="4.445" y2="50.8" width="0.6096" layer="1"/>
+<wire x1="4.445" y1="50.8" x2="3.683" y2="51.562" width="0.6096" layer="1"/>
 </signal>
 <signal name="N$2">

Commit message: Updated GSM Version
Parts:
- R_PROG: value 1.2KΩ=1A -> 1.2KΩ
- moved U$1 0.25 mm to (8.64, 54.6)
Other:
- board text added: "12-Jun-2016 Rev.04"
- board text removed: "12-Jun-2016 Rev.03"
Changed lines of the file:
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@@
 <rectangle x1="4.826" y1="61.0235" x2="8.255" y2="63.4365" layer="29"/>
 <hole x="2.0955" y="78.2955" drill="1.5"/>
-<text x="23.0505" y="59.7535" size="1.4224" layer="25" rot="R270" align="center">12-Jun-2016
-Rev.03</text>
-<text x="13.081" y="75.438" size="1.778" layer="25" rot="R90">ON</text>
-<text x="5.6515" y="74.422" size="1.778" layer="25" rot="R90">OFF</text>
+<text x="21.336" y="59.817" size="1.4224" layer="25" rot="R270" align="center">12-Jun-2016
+Rev.04</text>
+<text x="12.065" y="78.0415" size="1.27" layer="25" rot="R90" align="center">ON</text>
+<text x="4.318" y="78.105" size="1.27" layer="25" rot="R90" align="center">OFF</text>
 </plain>
 <attributes>
@@
 <elements>
 <element name="+" library="SparkFun-Connectors" package="1X02" value="BAT" x="2.032" y="73.5965" smashed="yes" rot="R270">
-<attribute name="NAME" x="1.1938" y="77.1017" size="1.6764" layer="25" ratio="10" rot="R270"/>
-<attribute name="VALUE" x="3.8735" y="73.406" size="1.27" layer="25" rot="R270"/>
+<attribute name="NAME" x="2.0193" y="76.0857" size="1.778" layer="25" ratio="10" rot="R270" align="center"/>
+<attribute name="VALUE" x="4.572" y="72.644" size="1.27" layer="25" rot="R270" align="center"/>
 </element>
 <element name="C1" library="resistor" package="C1206" value="10μf" x="9.3345" y="73.025" smashed="yes">
-<attribute name="NAME" x="8.31849375" y="74.42200625" size="1.27" layer="25"/>
-<attribute name="VALUE" x="7.365990625" y="70.485" size="1.27" layer="25"/>
+<attribute name="NAME" x="9.33449375" y="75.24750625" size="1.27" layer="25" align="center"/>
+<attribute name="VALUE" x="9.3345" y="73.025009375" size="0.8128" layer="25" rot="R270" align="center"/>
 </element>
 <element name="C2" library="resistor" package="C1206" value="10μf" x="2.0955" y="62.23" smashed="yes" rot="R90">
-<attribute name="NAME" x="2.2225" y="57.404" size="1.27" layer="25" rot="R90"/>
-<attribute name="VALUE" x="2.2225" y="65.2145" size="1.27" layer="25" rot="R90"/>
+<attribute name="NAME" x="2.0955" y="65.4685" size="1.27" layer="25" rot="R180" align="center"/>
+<attribute name="VALUE" x="2.0955" y="62.23" size="0.8128" layer="25" align="center"/>
 </element>
 <element name="TP4056" library="TP4056" package="SOP-8" value="TP4056" x="6.5405" y="62.23" smashed="yes" rot="R90">
-<attribute name="NAME" x="10.4775" y="58.801" size="1.27" layer="25" rot="R90"/>
+<attribute name="NAME" x="9.906" y="62.23" size="1.27" layer="25" rot="R90" align="center"/>
 </element>
 <element name="JST2" library="SparkFun-Connectors" package="JST-2-SMD" value="+" x="8.636" y="46.863" smashed="yes" rot="R180">
 <attribute name="PROD_ID" value="CONN-11443" x="8.636" y="46.863" size="1.778" layer="27" rot="R180" display="off"/>
-<attribute name="NAME" x="10.4775" y="46.4185" size="1.016" layer="25" rot="R180"/>
-<attribute name="VALUE" x="8.382" y="43.4975" size="1.4224" layer="25" rot="R180"/>
+<attribute name="NAME" x="8.6995" y="46.228" size="1.27" layer="25" rot="R180" align="center"/>
+<attribute name="VALUE" x="7.493" y="42.926" size="1.778" layer="25" rot="R180" align="center"/>
 </element>
 <element name="LED1" library="led" package="CHIPLED_1206" value="RED" x="33.401" y="70.2945" smashed="yes">
-<attribute name="NAME" x="29.7815" y="75.057" size="1.27" layer="25" rot="R270"/>
-<attribute name="VALUE" x="28.067" y="74.422" size="1.27" layer="25" rot="R270"/>
+<attribute name="NAME" x="30.48" y="72.7075" size="1.27" layer="25" rot="R270" align="center"/>
+<attribute name="VALUE" x="33.401" y="74.7395" size="1.27" layer="25" rot="R90" align="center"/>
 </element>
 <element name="LED2" library="led" package="CHIPLED_1206" value="GREEN" x="33.401" y="64.516" smashed="yes" rot="R180">
-<attribute name="NAME" x="30.4165" y="62.611" size="1.27" layer="25" rot="R90"/>
-<attribute name="VALUE" x="28.575" y="61.976" size="1.27" layer="25" rot="R90"/>
+<attribute name="NAME" x="29.4005" y="64.516" size="1.27" layer="25" rot="R90" align="center"/>
+<attribute name="VALUE" x="30.9245" y="64.516" size="1.016" layer="25" rot="R270" align="center"/>
 </element>
 <element name="R2" library="resistor" package="R1206" value="150Ω" x="30.5435" y="75.3745" smashed="yes" rot="MR180">
-<attribute name="NAME" x="31.369" y="72.644" size="1.27" layer="26" rot="MR180"/>
-<attribute name="VALUE" x="26.0985" y="72.644" size="1.27" layer="26" rot="MR180"/>
+<attribute name="NAME" x="30.5435" y="71.9455" size="1.27" layer="26" rot="MR180" align="center"/>
+<attribute name="VALUE" x="30.5435" y="75.3745" size="0.8128" layer="26" rot="MR270" align="center"/>
 </element>
 <element name="R3" library="resistor" package="R1206" value="150Ω" x="33.4645" y="54.991" smashed="yes" rot="R90">
-<attribute name="NAME" x="29.083" y="53.848" size="1.27" layer="25" rot="R90"/>
-<attribute name="VALUE" x="30.988" y="52.451" size="1.27" layer="25" rot="R90"/>
-</element>
-<element name="R_PROG" library="resistor" package="R1206" value="1.2KΩ=1A" x="4.826" y="56.8325" smashed="yes">
-<attribute name="NAME" x="1.5875" y="53.2765" size="1.27" layer="25"/>
-<attribute name="VALUE" x="10.033" y="53.213" size="1.27" layer="25"/>
+<attribute name="NAME" x="30.7975" y="54.991" size="1.27" layer="25" rot="R90" align="center"/>
+<attribute name="VALUE" x="33.4645" y="54.991" size="0.8128" layer="25" align="center"/>
+</element>
+<element name="R_PROG" library="resistor" package="R1206" value="1.2KΩ" x="4.826" y="56.8325" smashed="yes">
+<attribute name="NAME" x="4.826" y="53.721" size="1.016" layer="25" align="center"/>
+<attribute name="VALUE" x="4.826" y="56.769" size="0.8128" layer="25" rot="R270" align="center"/>
 </element>
 <element name="USB" library="micro usb B - sparkfun - china - hole 4LEGS TEST" package="MICRO_USB_4_LEGS" value="MICRO-USB-B" x="22.86" y="77.9145" smashed="yes" rot="MR270">
-<attribute name="NAME" x="20.7645" y="72.898" size="1.6764" layer="26" rot="MR180"/>
+<attribute name="NAME" x="22.86" y="71.8185" size="1.27" layer="26" rot="MR180" align="center"/>
 <attribute name="VALUE" x="21.209" y="72.7075" size="0.4064" layer="28" rot="MR180"/>
 </element>
@@
 <element name="WIXEL" library="wixel" package="WIXEL_PARAKEET_ONLY" value="WIXEL_PARAKEET_ONLY" x="22.86" y="62.23" smashed="yes"/>
 <element name="SIM800L" library="SIM800L Module" package="SIM800L_PARAKEET_ONLY" value="SIM800L_PARAKEET_ONLY" x="22.6695" y="62.865" smashed="yes" rot="MR180"/>
-<element name="U$1" library="LOGO" package="PARAKEET_VECTOR" value="" x="8.89" y="54.61" rot="MR0"/>
+<element name="U$1" library="LOGO" package="PARAKEET_VECTOR" value="" x="8.636" y="54.61" rot="MR0"/>
 </elements>
 <signals>

Commit message: Updated GSM Version
Parts:
- removed R3: 150Ω, resistor:R1206
- added R1: 330Ω, resistor:R1206
- R2: value 150Ω -> 330Ω
- moved R2 20.6 mm to (33.5, 55.0), flipped to the top, turned to 90 degrees
- moved C1 0.07 mm to (9.40, 73.1)
Connections:
- net GND: now also TP4056.9
- net N$3: now also R1.2; no longer R2.2
- net N$4: now also R2.2; no longer R3.2
- net N$5: now also R1.1; no longer R2.1
- net N$6: now also R2.1; no longer R3.1
Routing:
- net N$7: track 64.9 -> 65.5 mm
Other:
- board text added: "14-Jun-2016 Rev.05"
- board text removed: "12-Jun-2016 Rev.04"

Commit message: Updated GSM version
Parts:
- moved R_PROG 10.5 mm to (8.10, 46.8), flipped to the bottom
- moved C2 7.71 mm to (6.22, 55.7), turned to 180 degrees
- moved + 2.65 mm to (3.92, 71.7), turned to 90 degrees
- moved U$1 1.42 mm to (9.88, 55.3)
- moved SWITCH 0.94 mm to (9.07, 78.1)
- moved JST2 0.63 mm to (9.27, 46.9)
Routing:
- net N$1: track 3.35 -> 14.5 mm, vias 0 -> 1
- net N$8: track 51.9 -> 47.1 mm
- net N$7: track 65.5 -> 63.1 mm
- net N$3: track 6.02 -> 5.22 mm
Other:
- board size 35 x 38.4 mm -> 33.5 x 38.5 mm
- board text added: "14-Jun-2016 Rev.06"
- board text removed: "14-Jun-2016 Rev.05"
