File: Other Versions/GSM-Parakeet/parakeet_board_rev.07.brd (EAGLE design)
At the start: 33.5 x 38.5 mm, 15 parts

Commit message: Updated GSM version
Parts:
- LED1: value RED -> Red; device led:CHIPLED_1206 -> SparkFun-LED:LED-1206
- LED2: value GREEN -> Green; device led:CHIPLED_1206 -> SparkFun-LED:LED-1206
- moved U$1 3.26 mm to (9.82, 58.5)
- turned LED2 to 270 degrees
- turned LED1 to 90 degrees
Routing:
- net N$7: track 63.1 -> 63.6 mm
Other:
- board text added: "15-Jun-2016 Rev.07"
- board text removed: "14-Jun-2016 Rev.06"
