File: Other Versions/GSM-Parakeet/parakeet_board_rev.07.sch (EAGLE design)
At the start: 14 parts

Commit message: Updated GSM version
Parts:
- LED1: value RED -> Red; device led:LEDCHIPLED_1206 -> SparkFun-LED:LED1206
- LED2: value GREEN -> Green; device led:LEDCHIPLED_1206 -> SparkFun-LED:LED1206
Changed lines of the file:
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@@
 <part name="R_PROG" library="resistor" deviceset="R-EU_" device="R1206" value="1.2KΩ"/>
 <part name="C1" library="resistor" deviceset="C-EU" device="C1206" value="10μf"/>
-<part name="LED1" library="led" deviceset="LED" device="CHIPLED_1206" value="RED"/>
-<part name="LED2" library="led" deviceset="LED" device="CHIPLED_1206" value="GREEN"/>
 <part name="R1" library="resistor" deviceset="R-EU_" device="R1206" value="330Ω"/>
 <part name="R2" library="resistor" deviceset="R-EU_" device="R1206" value="330Ω"/>
@@
 <part name="WIXEL" library="wixel" deviceset="WIXEL_PARAKEET_ONLY" device=""/>
 <part name="SIM800L" library="SIM800L Module" deviceset="SIM800L_PARAKEET_ONLY" device=""/>
+<part name="LED1" library="SparkFun-LED" deviceset="LED" device="1206" value="Red"/>
+<part name="LED2" library="SparkFun-LED" deviceset="LED" device="1206" value="Green"/>
 </parts>
 <sheets>
@@
 <instance part="R_PROG" gate="G$1" x="22.86" y="43.18"/>
 <instance part="C1" gate="G$1" x="60.96" y="30.48" rot="R270"/>
-<instance part="LED1" gate="G$1" x="83.82" y="45.72" rot="R270"/>
-<instance part="LED2" gate="G$1" x="83.82" y="38.1" rot="R270"/>
 <instance part="R1" gate="G$1" x="71.12" y="45.72"/>
 <instance part="R2" gate="G$1" x="71.12" y="38.1"/>
@@
 <instance part="WIXEL" gate="G$1" x="121.92" y="40.64"/>
 <instance part="SIM800L" gate="G$1" x="157.48" y="40.64"/>
+<instance part="LED1" gate="G$1" x="83.82" y="45.72" rot="R270"/>
+<instance part="LED2" gate="G$1" x="83.82" y="38.1" rot="R270"/>
 </instances>
 <busses>
@@
 <net name="N$3" class="0">
 <segment>
-<pinref part="LED1" gate="G$1" pin="C"/>
 <pinref part="R1" gate="G$1" pin="2"/>
 <wire x1="76.2" y1="45.72" x2="78.74" y2="45.72" width="0.1524" layer="91"/>
+<pinref part="LED1" gate="G$1" pin="C"/>
 </segment>
 </net>
 <net name="N$4" class="0">
 <segment>
-<pinref part="LED2" gate="G$1" pin="C"/>
 <pinref part="R2" gate="G$1" pin="2"/>
 <wire x1="76.2" y1="38.1" x2="78.74" y2="38.1" width="0.1524" layer="91"/>
+<pinref part="LED2" gate="G$1" pin="C"/>
 </segment>
 </net>
@@
 <wire x1="63.5" y1="50.8" x2="86.36" y2="50.8" width="0.1524" layer="91"/>
 <wire x1="86.36" y1="50.8" x2="86.36" y2="45.72" width="0.1524" layer="91"/>
-<pinref part="LED1" gate="G$1" pin="A"/>
-<pinref part="LED2" gate="G$1" pin="A"/>
+<pinref part="TP4056" gate="G$1" pin="VCC"/>
 <wire x1="86.36" y1="45.72" x2="86.36" y2="38.1" width="0.1524" layer="91"/>
-<pinref part="TP4056" gate="G$1" pin="VCC"/>
 <wire x1="30.48" y1="38.1" x2="22.86" y2="38.1" width="0.1524" layer="91"/>
 <wire x1="22.86" y1="38.1" x2="22.86" y2="50.8" width="0.1524" layer="91"/>
@@
 <pinref part="C2" gate="G$1" pin="1"/>
 <junction x="22.86" y="38.1"/>
+<pinref part="LED1" gate="G$1" pin="A"/>
 <junction x="86.36" y="45.72"/>
+<pinref part="LED2" gate="G$1" pin="A"/>
 </segment>
 </net>
