File: Other Versions/GSM-Parakeet/parakeet_board_rev.08.brd (EAGLE design)
At the start: 33.5 x 38.5 mm, 15 parts

Commit message: Updated GSM Version
Parts:
- removed U$1: (no value), LOGO:PARAKEET_VECTOR
- added U$2: (no value), LOGO:PARAKEET
Other:
- board text added: "15-Jun-2016 Rev.08"
- board text removed: "15-Jun-2016 Rev.07"
Changed lines of the file:
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@@
 <layer number="21" name="tPlace" color="7" fill="1" visible="yes" active="yes"/>
 <layer number="22" name="bPlace" color="7" fill="1" visible="yes" active="yes"/>
-<layer number="23" name="tOrigins" color="15" fill="1" visible="no" active="yes"/>
-<layer number="24" name="bOrigins" color="15" fill="1" visible="no" active="yes"/>
+<layer number="23" name="tOrigins" color="15" fill="1" visible="yes" active="yes"/>
+<layer number="24" name="bOrigins" color="15" fill="1" visible="yes" active="yes"/>
 <layer number="25" name="tNames" color="7" fill="1" visible="yes" active="yes"/>
 <layer number="26" name="bNames" color="7" fill="1" visible="yes" active="yes"/>
@@
 <hole x="3.62125" y="78.27405625" drill="1.5"/>
 <text x="21.336" y="59.817" size="1.4224" layer="25" rot="R270" align="center">15-Jun-2016
-Rev.07</text>
+Rev.08</text>
 <text x="12.065" y="78.0415" size="1.27" layer="25" rot="R90" align="center">ON</text>
 <text x="6.089484375" y="78.183221875" size="1.27" layer="25" rot="R90" align="center">OFF</text>
@@
 <param name="mvStopFrame" value="1"/>
 <param name="mvCreamFrame" value="0"/>
-<param name="mlMinStopFrame" value="3mil"/>
-<param name="mlMaxStopFrame" value="3mil"/>
+<param name="mlMinStopFrame" value="2.5mil"/>
+<param name="mlMaxStopFrame" value="2.5mil"/>
 <param name="mlMinCreamFrame" value="0mil"/>
 <param name="mlMaxCreamFrame" value="0mil"/>
@@
 <element name="WIXEL" library="wixel" package="WIXEL_PARAKEET_ONLY" value="WIXEL_PARAKEET_ONLY" x="22.86" y="62.23" smashed="yes"/>
 <element name="SIM800L" library="SIM800L Module" package="SIM800L_PARAKEET_ONLY" value="SIM800L_PARAKEET_ONLY" x="22.6695" y="62.865" smashed="yes" rot="MR180"/>
-<element name="U$1" library="LOGO" package="PARAKEET_VECTOR" value="" x="9.8220375" y="58.54895625" rot="MR0"/>
 <element name="LED1" library="SparkFun-LED" package="LED-1206" value="Red" x="33.410953125" y="70.292546875" smashed="yes" rot="R90">
 <attribute name="NAME" x="30.96075" y="73.26073125" size="1.27" layer="25" rot="R90" align="center"/>
@@
 <attribute name="VALUE" x="30.9224" y="64.844565625" size="1.27" layer="25" rot="R270" align="center"/>
 </element>
+<element name="U$2" library="LOGO" package="PARAKEET" value="" x="9.896709375" y="58.539990625" rot="MR0"/>
 </elements>
 <signals>
@@
 <contactref element="JST2" pad="1"/>
 <contactref element="+" pad="2"/>
-<polygon width="0.2" layer="1">
+<polygon width="0.2" layer="1" isolate="0.254">
 <vertex x="-3.81" y="85.09"/>
 <vertex x="40.64" y="85.09"/>
@@
 <vertex x="-3.81" y="36.83"/>
 </polygon>
-<polygon width="0.2" layer="16">
+<polygon width="0.2" layer="16" isolate="0.254">
 <vertex x="-1.27" y="82.55"/>
 <vertex x="38.1" y="82.55"/>
@@
 <contactref element="SIM800L" pad="P$6_GND"/>
 <contactref element="TP4056" pad="9"/>
-<via x="22.779771875" y="76.395359375" extent="1-16" drill="0.3302"/>
-<via x="25.082325" y="74.59676875" extent="1-16" drill="0.3302"/>
+<via x="22.779771875" y="76.371853125" extent="1-16" drill="0.3302"/>
+<via x="25.02078125" y="74.63010625" extent="1-16" drill="0.3302"/>
 <via x="24.147834375" y="73.105246875" extent="1-16" drill="0.3302"/>
 <via x="13.187675" y="72.278246875" extent="1-16" drill="0.3302"/>
@@
 <via x="4.189215625" y="66.5624125" extent="1-16" drill="0.3302"/>
 <via x="4.097240625" y="62.257740625" extent="1-16" drill="0.3302"/>
-<via x="7.33674375" y="58.064028125" extent="1-16" drill="0.3302"/>
+<via x="7.3952125" y="58.10403125" extent="1-16" drill="0.3302"/>
 <via x="9.570896875" y="44.686021875" extent="1-16" drill="0.3302"/>
 <via x="24.349728125" y="51.50676875" extent="1-16" drill="0.3302"/>
@@
 <via x="28.6529625" y="77.44675625" extent="1-16" drill="0.3302"/>
 <via x="16.268671875" y="52.5453125" extent="1-16" drill="0.3302"/>
-<via x="3.820909375" y="58.303246875" extent="1-16" drill="0.3302"/>
+<via x="3.87005625" y="58.3652125" extent="1-16" drill="0.3302"/>
 <via x="33.51016875" y="46.95656875" extent="1-16" drill="0.3302"/>
 <via x="3.689540625" y="47.332578125" extent="1-16" drill="0.3302"/>
@@
 <signal name="N$3">
 <contactref element="R1" pad="2"/>
-<via x="34.152125" y="74.33583125" extent="1-16" drill="0.6"/>
-<wire x1="34.152125" y1="72.795625" x2="34.152125" y2="74.33583125" width="0.7" layer="1"/>
-<wire x1="34.152125" y1="74.33583125" x2="33.11345625" y2="75.3745" width="0.7" layer="16"/>
-<wire x1="33.11345625" y1="75.3745" x2="31.9655" y2="75.3745" width="0.7" layer="16"/>
+<via x="34.037240625" y="74.31285625" extent="1-16" drill="0.6"/>
 <contactref element="LED1" pad="C"/>
-<wire x1="33.410953125" y1="71.792546875" x2="33.410953125" y2="72.054453125" width="0.7" layer="1"/>
-<wire x1="33.410953125" y1="72.054453125" x2="34.152125" y2="72.795625" width="0.7" layer="1"/>
+<wire x1="33.410953125" y1="71.792546875" x2="34.037240625" y2="72.418834375" width="0.7" layer="1"/>
+<wire x1="34.037240625" y1="72.418834375" x2="34.037240625" y2="74.31285625" width="0.7" layer="1"/>
+<wire x1="34.037240625" y1="74.31285625" x2="32.975596875" y2="75.3745" width="0.7" layer="16"/>
+<wire x1="32.975596875" y1="75.3745" x2="31.9655" y2="75.3745" width="0.7" layer="16"/>
 </signal>
 <signal name="N$4">
@@
 </signal>
 <signal name="N$10">
-<polygon width="0.4064" layer="16" pour="cutout">
+<polygon width="0.002540625" layer="16" pour="cutout">
 <vertex x="31.75" y="41.91"/>
 <vertex x="31.75" y="49.53"/>
@@
 </signal>
 <signal name="N$11">
-<polygon width="0.4064" layer="1" pour="cutout">
+<polygon width="0.002540625" layer="1" pour="cutout">
 <vertex x="31.75" y="41.91"/>
 <vertex x="13.97" y="41.91"/>
