File: Other Versions/GSM-Parakeet/parakeet_board_rev.1.0.sch (EAGLE design)
At the start: 14 parts

Commit message: updated parakeet version
Parts:
- removed +: BAT, SparkFun-Connectors:M02PTH
- added JST-XH: 2_PIN_JST-XH-B2B, JST-XH_HEADERS:2_PIN_JST-XH-B2B
Connections:
- net GND: now also JST-XH.P$2; no longer +.2
- net N$8: now also JST-XH.P$1; no longer +.1
Changed lines of the file:
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@@
 <part name="R2" library="resistor" deviceset="R-EU_" device="R1206" value="330Ω"/>
 <part name="C2" library="resistor" deviceset="C-EU" device="C1206" value="10μf"/>
-<part name="+" library="SparkFun-Connectors" deviceset="M02" device="PTH" value="BAT"/>
 <part name="JST2" library="SparkFun-Connectors" deviceset="M02" device="-JST-2MM-SMT" value="+"/>
 <part name="SWITCH" library="MSK-12C02 SMD Micro Slider Switch SPDT" deviceset="MSK-12C02_SMD_SPDT_SWITCH" device=""/>
@@
 <part name="LED1" library="SparkFun-LED" deviceset="LED" device="1206" value="Red"/>
 <part name="LED2" library="SparkFun-LED" deviceset="LED" device="1206" value="Green"/>
+<part name="JST-XH" library="JST-XH_HEADERS" deviceset="2_PIN_JST-XH-B2B" device=""/>
 </parts>
 <sheets>
@@
 <instance part="R2" gate="G$1" x="71.12" y="38.1"/>
 <instance part="C2" gate="G$1" x="22.86" y="35.56"/>
-<instance part="+" gate="G$1" x="101.6" y="33.02" rot="R180"/>
 <instance part="JST2" gate="G$1" x="101.6" y="48.26" rot="R180"/>
 <instance part="SWITCH" gate="MSK-12C02" x="102.87" y="60.96"/>
@@
 <instance part="LED1" gate="G$1" x="83.82" y="45.72" rot="R270"/>
 <instance part="LED2" gate="G$1" x="83.82" y="38.1" rot="R270"/>
+<instance part="JST-XH" gate="G$1" x="103.124" y="31.75" rot="R270"/>
 </instances>
 <busses>
@@
 <wire x1="93.98" y1="45.72" x2="91.44" y2="45.72" width="0.1524" layer="91"/>
 <wire x1="91.44" y1="45.72" x2="91.44" y2="30.48" width="0.1524" layer="91"/>
-<pinref part="+" gate="G$1" pin="2"/>
 <wire x1="91.44" y1="30.48" x2="91.44" y2="25.4" width="0.1524" layer="91"/>
-<wire x1="93.98" y1="30.48" x2="91.44" y2="30.48" width="0.1524" layer="91"/>
+<wire x1="93.98" y1="30.48" x2="93.726" y2="30.48" width="0.1524" layer="91"/>
 <junction x="91.44" y="30.48"/>
 <junction x="22.86" y="30.48"/>
 <pinref part="TP4056" gate="G$1" pin="GND_PAD"/>
 <junction x="46.99" y="30.48"/>
+<pinref part="JST-XH" gate="G$1" pin="P$2"/>
+<wire x1="93.726" y1="30.48" x2="91.44" y2="30.48" width="0.1524" layer="91"/>
+<junction x="93.726" y="30.48"/>
 </segment>
 <segment>
@@
 <wire x1="88.9" y1="33.02" x2="88.9" y2="48.26" width="0.1524" layer="91"/>
 <wire x1="88.9" y1="48.26" x2="93.98" y2="48.26" width="0.1524" layer="91"/>
-<pinref part="+" gate="G$1" pin="1"/>
-<wire x1="93.98" y1="33.02" x2="88.9" y2="33.02" width="0.1524" layer="91"/>
+<wire x1="93.98" y1="33.02" x2="93.726" y2="33.02" width="0.1524" layer="91"/>
 <junction x="88.9" y="33.02"/>
 <pinref part="SWITCH" gate="MSK-12C02" pin="COM"/>
+<wire x1="93.726" y1="33.02" x2="88.9" y2="33.02" width="0.1524" layer="91"/>
 <wire x1="95.25" y1="60.96" x2="88.9" y2="60.96" width="0.1524" layer="91"/>
 <wire x1="88.9" y1="60.96" x2="88.9" y2="48.26" width="0.1524" layer="91"/>
 <junction x="88.9" y="48.26"/>
+<pinref part="JST-XH" gate="G$1" pin="P$1"/>
+<junction x="93.726" y="33.02"/>
 </segment>
 </net>
